File: Esquematicos/Vumetro/Vumetro.sch (KiCad schematic (older format))
At the start: 19 parts, among them J1 AudioJack5_Ground, J2 Conn_Teclado_Matricial_4x4, P1 conn_pin40, P2 conn_pin40, U1 MAX7219, U2 conn_pin8, U3 conn_pin8, U4 opa2350pa

Commit message: Se modifica esquematico
Parts:
- C1: symbol Vumetro-rescue:C-Device -> Vumetro-rescue:C-Device-Vumetro-rescue
- C2: value 1.8 nF -> 2.2 nF; symbol Vumetro-rescue:C-Device -> Vumetro-rescue:C-Device-Vumetro-rescue
- C3, C4: symbol Vumetro-rescue:CAP-pspice -> Vumetro-rescue:CAP-pspice-Vumetro-rescue
- J1: symbol Vumetro-rescue:AudioJack5_Ground-Connector -> Vumetro-rescue:AudioJack5_Ground-Connector-Vumetro-rescue
- P1, P2: symbol Vumetro-rescue:conn_pin40-vumetro -> Vumetro-rescue:conn_pin40-vumetro-Vumetro-rescue
- R1, R2, R3, R4, R5, R6: symbol Vumetro-rescue:R-Device -> Vumetro-rescue:R-Device-Vumetro-rescue
- RV1: symbol Vumetro-rescue:R_POT-Device -> Vumetro-rescue:R_POT-Device-Vumetro-rescue
- U1: symbol Vumetro-rescue:MAX7219-vumetro -> Vumetro-rescue:MAX7219-vumetro-Vumetro-rescue
- U2, U3: symbol Vumetro-rescue:conn_pin8-vumetro-Vumetro-rescue-Vumetro-rescue -> Vumetro-rescue:conn_pin8-vumetro-Vumetro-rescue-Vumetro-rescue-Vumetro-rescue
- U4: symbol Vumetro-rescue:opa2350pa-vumetro-Vumetro-rescue-Vumetro-rescue -> Vumetro-rescue:opa2350pa-vumetro-Vumetro-rescue-Vumetro-rescue-Vumetro-rescue
Connections:
- net labels added: COL0, COL1, COL2, COL3, COL4, COL5, COL6, COL7, GPIO0, ROW0, ROW1, ROW2, ROW3, ROW4, ROW5, ROW6, ROW7
- net labels removed: DIC0, DIC1, DIC2, DIC3, DIC4, DIC5, DIC6, DIC7, SEGA, SEGB, SEGC, SEGD, SEGDP, SEGE, SEGF, SEGG
- wire segments 154 -> 155
- no-connect marks 46 -> 45
Changed lines of the file:
@@
 EESchema Schematic File Version 4
 LIBS:Vumetro-cache
-EELAYER 26 0
+EELAYER 29 0
 EELAYER END
 $Descr A4 11693 8268
@@
 $EndDescr
 $Comp
-L Vumetro-rescue:R-Device R1
+L Vumetro-rescue:R-Device-Vumetro-rescue R1
 U 1 1 5BD08240
 P 3350 2400
@@
 $EndComp
 $Comp
-L Vumetro-rescue:R-Device R2
+L Vumetro-rescue:R-Device-Vumetro-rescue R2
 U 1 1 5BD082FA
 P 3350 2900
@@
 $EndComp
 $Comp
-L Vumetro-rescue:GNDA-power #PWR0102
+L Vumetro-rescue:GNDA-power-Vumetro-rescue #PWR0102
 U 1 1 5BD08B01
 P 3600 1000
@@
 	2400 1400 1950 1400
 $Comp
-L Vumetro-rescue:R_POT-Device RV1
+L Vumetro-rescue:R_POT-Device-Vumetro-rescue RV1
 U 1 1 5BD09203
 P 2800 1650
@@
 Connection ~ 3350 2650
 $Comp
-L Vumetro-rescue:GNDA-power #PWR0103
+L Vumetro-rescue:GNDA-power-Vumetro-rescue #PWR0103
 U 1 1 5BD0D7F2
 P 3350 3200
@@
 $EndComp
 $Comp
-L Vumetro-rescue:C-Device C2
+L Vumetro-rescue:C-Device-Vumetro-rescue C2
 U 1 1 5BD1B29A
 P 4250 2900
 F 0 "C2" H 4365 2946 50  0000 L CNN
-F 1 "1.8 nF" H 4365 2855 50  0000 L CNN
+F 1 "2.2 nF" H 4365 2855 50  0000 L CNN
 F 2 "" H 4288 2750 50  0001 C CNN
 F 3 "~" H 4250 2900 50  0001 C CNN
@@
 $EndComp
 $Comp
-L Vumetro-rescue:GNDA-power #PWR0104
+L Vumetro-rescue:GNDA-power-Vumetro-rescue #PWR0104
 U 1 1 5BD1B343
 P 4250 3200
@@
 	4250 3050 4250 3200
 $Comp
-L Vumetro-rescue:R-Device R4
+L Vumetro-rescue:R-Device-Vumetro-rescue R4
 U 1 1 5BD1B49E
 P 3750 2650
@@
 Connection ~ 4250 2650
 $Comp
-L Vumetro-rescue:R-Device R5
+L Vumetro-rescue:R-Device-Vumetro-rescue R5
 U 1 1 5BD1FFCF
 P 4250 1800
@@
 $EndComp
 $Comp
-L Vumetro-rescue:R-Device R6
+L Vumetro-rescue:R-Device-Vumetro-rescue R6
 U 1 1 5BD204D6
 P 4700 1500
@@
 	4250 1500 4250 1650
 $Comp
-L Vumetro-rescue:GNDA-power #PWR0105
+L Vumetro-rescue:GNDA-power-Vumetro-rescue #PWR0105
 U 1 1 5BD20C9D
 P 4250 2200
@@
 	4250 1950 4250 2200
 $Comp
-L Vumetro-rescue:C-Device C1
+L Vumetro-rescue:C-Device-Vumetro-rescue C1
 U 1 1 5BD214BE
 P 2800 2200
@@
 CH1
 $Comp
-L Vumetro-rescue:conn_pin8-vumetro-Vumetro-rescue-Vumetro-rescue U2
+L Vumetro-rescue:conn_pin8-vumetro-Vumetro-rescue-Vumetro-rescue-Vumetro-rescue U2
 U 1 1 5BD8D993
 P 4200 3850
@@
 $EndComp
 $Comp
-L Vumetro-rescue:conn_pin8-vumetro-Vumetro-rescue-Vumetro-rescue U3
+L Vumetro-rescue:conn_pin8-vumetro-Vumetro-rescue-Vumetro-rescue-Vumetro-rescue U3
 U 1 1 5BD8E115
 P 4650 3850
@@
 $EndComp
 $Comp
-L Vumetro-rescue:opa2350pa-vumetro-Vumetro-rescue-Vumetro-rescue U4
+L Vumetro-rescue:opa2350pa-vumetro-Vumetro-rescue-Vumetro-rescue-Vumetro-rescue U4
 U 1 1 5BD9369A
 P 5350 2250
@@
 	4250 1050 4250 1500
 $Comp
-L Vumetro-rescue:GNDA-power #PWR0106
+L Vumetro-rescue:GNDA-power-Vumetro-rescue #PWR0106
 U 1 1 5BD9D42A
 P 4850 2900
@@
 	1300 4050 3250 4050
 Text Label 3250 4750 0    50   ~ 0
-DIC0
+ROW0
 Text Label 3800 4050 0    50   ~ 0
-DIC0
+ROW4
 Wire Wire Line
 	3800 4050 4000 4050
@@
 	4000 4750 3800 4750
 Text Label 3250 4550 0    50   ~ 0
-DIC6
+ROW6
 Text Label 3250 4450 0    50   ~ 0
-DIC2
+ROW2
 Text Label 3250 4350 0    50   ~ 0
-DIC3
+ROW3
 Text Label 3250 4150 0    50   ~ 0
-DIC5
+ROW5
 Text Label 3250 4050 0    50   ~ 0
-DIC1
+ROW1
 Text Label 3800 4150 0    50   ~ 0
-DIC1
+ROW6
 Text Label 3800 4250 0    50   ~ 0
-DIC2
+COL1
 Text Label 3800 4350 0    50   ~ 0
-DIC3
+COL2
 Text Label 3800 4450 0    50   ~ 0
-DIC4
+ROW7
 Text Label 3800 4550 0    50   ~ 0
-DIC5
+COL4
 Text Label 3800 4650 0    50   ~ 0
-DIC6
+ROW5
 Text Label 3800 4750 0    50   ~ 0
-DIC7
+ROW2
 Wire Wire Line
 	5300 5450 5300 4950
@@
 	3200 6250 6500 6250
 Text Label 5100 5150 1    50   ~ 0
-SEGD
+COL3
 Text Label 5300 5200 1    50   ~ 0
-SEGDP
+COL7
 Text Label 5500 5150 1    50   ~ 0
-SEGE
+COL2
 Text Label 5700 5150 1    50   ~ 0
-SEGC
+COL4
 Text Label 5900 5150 1    50   ~ 0
-SEGG
+COL0
 Text Label 6100 5150 1    50   ~ 0
-SEGB
+COL5
 Text Label 6300 5150 1    50   ~ 0
-SEGF
+COL1
 Text Label 6500 5150 1    50   ~ 0
-SEGA
+COL6
 Wire Wire Line
 	4850 4750 5100 4750
@@
 	4850 4050 5100 4050
 Text Label 5100 4050 0    50   ~ 0
-SEGDP
+COL7
 Text Label 5100 4150 0    50   ~ 0
-SEGA
+COL6
 Text Label 5100 4250 0    50   ~ 0
-SEGB
+ROW1
 Text Label 5100 4350 0    50   ~ 0
-SEGC
+COL0
 Text Label 5100 4450 0    50   ~ 0
-SEGD
+ROW3
 Text Label 5100 4550 0    50   ~ 0
-SEGE
+COL5
 Text Label 5100 4650 0    50   ~ 0
-SEGF
+COL3
 Text Label 5100 4750 0    50   ~ 0
-SEGG
+ROW0
 Wire Wire Line
 	2200 5550 1950 5550
 Wire Wire Line
 	2200 6050 1950 6050
-Text Label 1950 5550 0    50   ~ 0
-GND
 Text Label 1950 6050 0    50   ~ 0
-GND
+GNDA
 Wire Wire Line
 	3200 5850 3350 5850
@@
 ISET
 $Comp
-L Vumetro-rescue:CAP-pspice C4
+L Vumetro-rescue:CAP-pspice-Vumetro-rescue C4
 U 1 1 5BDF9589
 P 4900 6800
@@
 $EndComp
 $Comp
-L Vumetro-rescue:CAP-pspice C3
+L Vumetro-rescue:CAP-pspice-Vumetro-rescue C3
 U 1 1 5BDF96A7
 P 4300 6800
@@
 $EndComp
 $Comp
-L Vumetro-rescue:R-Device R3
+L Vumetro-rescue:R-Device-Vumetro-rescue R3
 U 1 1 5BDF9744
 P 3600 7050
@@
 $EndComp
 $Comp
-L Vumetro-rescue:GNDA-power #PWR0107
+L Vumetro-rescue:GNDA-power-Vumetro-rescue #PWR0107
 U 1 1 5BDF9885
 P 4300 7150
@@
 $EndComp
 $Comp
-L Vumetro-rescue:+5V-power #PWR0108
+L Vumetro-rescue:+5V-power-Vumetro-rescue #PWR0108
 U 1 1 5BDFBFF0
 P 3800 6550
@@
 $EndComp
 $Comp
-L Vumetro-rescue:GNDA-power #PWR0109
+L Vumetro-rescue:GNDA-power-Vumetro-rescue #PWR0109
 U 1 1 5BDFC0B2
 P 4900 7150
@@
 	2200 6350 1950 6350
 Text Label 1950 6350 0    50   ~ 0
-GND
+GPIO0
 Wire Wire Line
 	2200 5250 2100 5250
@@
 NoConn ~ 3200 5250
 $Comp
-L Vumetro-rescue:AudioJack5_Ground-Connector J1
+L Vumetro-rescue:AudioJack5_Ground-Connector-Vumetro-rescue J1
 U 1 1 5BE5F8BB
 P 1750 1200
@@
 NoConn ~ 1950 1100
 $Comp
-L Vumetro-rescue:conn_pin40-vumetro P2
-U 1 1 5BD92927
-P 8250 2750
-F 0 "P2" H 8250 2815 50  0000 C CNN
-F 1 "conn_pin40" H 8250 2724 50  0000 C CNN
-F 2 "" H 8250 2750 50  0001 C CNN
-F 3 "" H 8250 2750 50  0001 C CNN
-	1    8250 2750
-	1    0    0    -1
-$EndComp
-$Comp
-L Vumetro-rescue:conn_pin40-vumetro P1
+L Vumetro-rescue:conn_pin40-vumetro-Vumetro-rescue P1
 U 1 1 5BD936AB
 P 9700 2750
@@
 NoConn ~ 8000 3850
 NoConn ~ 8000 4050
-NoConn ~ 8000 4350
 NoConn ~ 8000 4450
 NoConn ~ 8000 4550
@@
 	4950 1050 4950 2450
 $Comp
-L Vumetro-rescue:PWR_FLAG-power #FLG0101
+L Vumetro-rescue:PWR_FLAG-power-Vumetro-rescue #FLG0101
 U 1 1 5C0A1FED
 P 1050 1900
@@
 	1900 4650 3250 4650
 Text Label 3250 4650 0    50   ~ 0
-DIC4
+ROW4
 Wire Wire Line
 	2200 5950 1500 5950
@@
 	1500 4250 3250 4250
 Text Label 3250 4250 0    50   ~ 0
-DIC7
-$Comp
-L Vumetro-rescue:MAX7219-vumetro U1
+ROW7
+$Comp
+L Vumetro-rescue:MAX7219-vumetro-Vumetro-rescue U1
 U 1 1 5BD94EE9
 P 2700 5150
@@
 $EndComp
 $Comp
-L Vumetro-rescue:PWR_FLAG-power #FLG0102
+L Vumetro-rescue:PWR_FLAG-power-Vumetro-rescue #FLG0102
 U 1 1 5BDCD5F1
 P 1050 3000
@@
 $EndComp
 $Comp
-L Vumetro-rescue:GNDA-power #PWR0110
+L Vumetro-rescue:GNDA-power-Vumetro-rescue #PWR0110
 U 1 1 5BE11156
 P 1050 1900
@@
 $EndComp
 $Comp
-L Vumetro-rescue:PWR_FLAG-power #FLG0103
+L Vumetro-rescue:PWR_FLAG-power-Vumetro-rescue #FLG0103
 U 1 1 5BE11DF9
 P 1050 2450
@@
 $EndComp
 $Comp
-L Vumetro-rescue:+5V-power #PWR0111
+L Vumetro-rescue:+5V-power-Vumetro-rescue #PWR0111
 U 1 1 5BE126C5
 P 1050 2450
@@
 	3350 2250 3350 2050
 $Comp
-L Vumetro-rescue:+3V3-power #PWR0112
+L Vumetro-rescue:+3V3-power-Vumetro-rescue #PWR0112
 U 1 1 5BDC2B19
 P 3350 2050
@@
 	5750 2450 6050 2450
 $Comp
-L Vumetro-rescue:+3V3-power #PWR0101
+L Vumetro-rescue:+3V3-power-Vumetro-rescue #PWR0101
 U 1 1 5BDC0419
 P 1050 3000
@@
 $EndComp
 $Comp
-L Vumetro-rescue:+3V3-power #PWR0113
+L Vumetro-rescue:+3V3-power-Vumetro-rescue #PWR0113
 U 1 1 5BDD5FCB
 P 6050 2150
@@
 Text Label 9250 4150 2    50   ~ 0
 232_TX
+$Comp
+L Vumetro-rescue:conn_pin40-vumetro-Vumetro-rescue P2
+U 1 1 5BD92927
+P 8250 2750
+F 0 "P2" H 8250 2815 50  0000 C CNN
+F 1 "conn_pin40" H 8250 2724 50  0000 C CNN
+F 2 "" H 8250 2750 50  0001 C CNN
+F 3 "" H 8250 2750 50  0001 C CNN
+	1    8250 2750
+	1    0    0    -1
+$EndComp
+Wire Wire Line
+	8000 4350 7650 4350
+Text Label 7650 4350 0    50   ~ 0
+GPIO0
+Text Label 1950 5550 0    50   ~ 0
+GNDA
 $EndSCHEMATC
